Commit message: Added a error finder node error_calibration to publich error left

File: ABBRobots/IRB6640/irb6640_ros2_gazebo/urdf/irb6640_camera.urdf.xacro (robot description, xacro)
@@ -5,5 +5,5 @@
             <parent link="${prefix}tool0"/>
             <child link="${prefix}camera_link"/>
-            <origin xyz="0.0 0 0.01" rpy="0 -1.57 0"/>
+            <origin xyz="0.0 0.0 0.0" rpy="0 -1.57 0"/>
         </joint>
         <link name="${prefix}camera_link">
